Commit message: Added cylinder, IIWA rotated 180deg, grid with 6 spaces.

File: public/drake_models/iiwa_description/urdf/iiwa7.urdf (robot description, URDF)
Before this commit: robot iiwa7, 9 links, 8 joints
Joints:
- joint iiwa_joint_6: origin xyz=0 -0.060700 0.2155 rpy=0 0 0 -> xyz=0 0.060700 0.2155 rpy=0 0 0
- joint iiwa_joint_7: origin xyz=0 0.060700 0.0805 rpy=0 0 0 -> xyz=0 -0.060700 0.0805 rpy=0 0 0

Commit message: Removed limits from the URDF. Make the arms move.

File: public/drake_models/iiwa_description/urdf/iiwa7.urdf (robot description, URDF)
Before this commit: robot iiwa7, 9 links, 8 joints
Joints:
- joint iiwa_joint_1: type revolute -> continuous
- joint iiwa_joint_2: type revolute -> continuous
- joint iiwa_joint_3: type revolute -> continuous
- joint iiwa_joint_4: type revolute -> continuous
- joint iiwa_joint_5: type revolute -> continuous
- joint iiwa_joint_6: type revolute -> continuous
- joint iiwa_joint_7: type revolute -> continuous

Commit message: Updated some reference frames in the URDF.

File: public/drake_models/iiwa_description/urdf/iiwa7.urdf (robot description, URDF)
Before this commit: robot iiwa7, 9 links, 8 joints
Joints:
- joint iiwa_joint_4: axis 0 -1 0 -> 0 1 0
- joint iiwa_joint_6: axis 0 1 0 -> 0 -1 0; origin xyz=0 0.060700 0.2155 rpy=0 0 0 -> xyz=0 -0.060700 0.2155 rpy=0 0 0
- joint iiwa_joint_7: origin xyz=0 -0.060700 0.0805 rpy=0 0 0 -> xyz=0 0.060700 0.0805 rpy=0 0 0

Commit message: Updated trajectory format. Using only one scene panel.

File: public/drake_models/iiwa_description/urdf/iiwa7.urdf (robot description, URDF)
Before this commit: robot iiwa7, 9 links, 8 joints
Joints:
- removed joint iiwa_joint_1
- removed joint iiwa_joint_2
- removed joint iiwa_joint_3
- removed joint iiwa_joint_4
- removed joint iiwa_joint_5
- removed joint iiwa_joint_6
- removed joint iiwa_joint_7
- added joint iiwa_joint1: type continuous, parent iiwa_link_0, child iiwa_link_1, origin xyz=0 0 0.1575 rpy=0 0 0, axis 0 0 1
- added joint iiwa_joint2: type continuous, parent iiwa_link_1, child iiwa_link_2, origin xyz=0 0 0.183 rpy=0 0 0, axis 0 1 0
- added joint iiwa_joint3: type continuous, parent iiwa_link_2, child iiwa_link_3, origin xyz=0 0 0.183 rpy=0 0 0, axis 0 0 1
- added joint iiwa_joint4: type continuous, parent iiwa_link_3, child iiwa_link_4, origin xyz=0 0 0.2155 rpy=0 0 0, axis 0 1 0
- added joint iiwa_joint5: type continuous, parent iiwa_link_4, child iiwa_link_5, origin xyz=0 0 0.184 rpy=0 0 0, axis 0 0 1
- added joint iiwa_joint6: type continuous, parent iiwa_link_5, child iiwa_link_6, origin xyz=0 -0.060700 0.2155 rpy=0 0 0, axis 0 -1 0
- added joint iiwa_joint7: type continuous, parent iiwa_link_6, child iiwa_link_7, origin xyz=0 0.060700 0.0805 rpy=0 0 0, axis 0 0 1
