Commit message: Iiwa joints renamed from 0 to 6.

File: public/models/iiwa/urdf/iiwa7.urdf (robot description, URDF)
Before this commit: robot iiwa7, 9 links, 8 joints
Joints:
- removed joint iiwa_joint7
- added joint iiwa_joint0: type continuous, parent iiwa_link_0, child iiwa_link_1, origin xyz=0 0 0.1575 rpy=0 0 0, axis 0 0 1
- joint iiwa_joint1: axis 0 0 1 -> 0 1 0; child iiwa_link_1 -> iiwa_link_2; origin xyz=0 0 0.1575 rpy=0 0 0 -> xyz=0 0 0.183 rpy=0 0 0; parent iiwa_link_0 -> iiwa_link_1
- joint iiwa_joint2: axis 0 1 0 -> 0 0 1; child iiwa_link_2 -> iiwa_link_3; parent iiwa_link_1 -> iiwa_link_2
- joint iiwa_joint3: axis 0 0 1 -> 0 1 0; child iiwa_link_3 -> iiwa_link_4; origin xyz=0 0 0.183 rpy=0 0 0 -> xyz=0 0 0.2155 rpy=0 0 0; parent iiwa_link_2 -> iiwa_link_3
- joint iiwa_joint4: axis 0 1 0 -> 0 0 1; child iiwa_link_4 -> iiwa_link_5; origin xyz=0 0 0.2155 rpy=0 0 0 -> xyz=0 0 0.184 rpy=0 0 0; parent iiwa_link_3 -> iiwa_link_4
- joint iiwa_joint5: axis 0 0 1 -> 0 -1 0; child iiwa_link_5 -> iiwa_link_6; origin xyz=0 0 0.184 rpy=0 0 0 -> xyz=0 -0.060700 0.2155 rpy=0 0 0; parent iiwa_link_4 -> iiwa_link_5
- joint iiwa_joint6: axis 0 -1 0 -> 0 0 1; child iiwa_link_6 -> iiwa_link_7; origin xyz=0 -0.060700 0.2155 rpy=0 0 0 -> xyz=0 0.060700 0.0805 rpy=0 0 0; parent iiwa_link_5 -> iiwa_link_6
