Commit message: Adding Allegro Hand urdf and mesh.

File: public/models/allegro/urdf/allegro_right_hand.urdf (robot description, URDF)
Before this commit: robot allegro_hand_right, 22 links, 21 joints
Links:
- link link_0: geometry visual mesh filename=../meshes/visual/link_0.stl
- link link_1: geometry visual mesh filename=../meshes/visual/link_1.stl
- link link_10: geometry visual mesh filename=../meshes/visual/link_2.stl
- link link_11: geometry visual mesh filename=../meshes/visual/link_3.stl
- link link_11_tip: geometry visual mesh filename=../meshes/visual/link_3_tip.stl
- link link_12: geometry visual mesh filename=../meshes/visual/link_12_right.stl
- link link_13: geometry visual mesh filename=../meshes/visual/link_13.stl
- link link_14: geometry visual mesh filename=../meshes/visual/link_14.stl
- link link_15: geometry visual mesh filename=../meshes/visual/link_15.stl
- link link_15_tip: geometry visual mesh filename=../meshes/visual/link_15_tip.stl
- link link_2: geometry visual mesh filename=../meshes/visual/link_2.stl
- link link_3: geometry visual mesh filename=../meshes/visual/link_3.stl
- link link_3_tip: geometry visual mesh filename=../meshes/visual/link_3_tip.stl
- link link_4: geometry visual mesh filename=../meshes/visual/link_0.stl
- link link_5: geometry visual mesh filename=../meshes/visual/link_1.stl
- link link_6: geometry visual mesh filename=../meshes/visual/link_2.stl
- link link_7: geometry visual mesh filename=../meshes/visual/link_3.stl
- link link_7_tip: geometry visual mesh filename=../meshes/visual/link_3_tip.stl
- link link_8: geometry visual mesh filename=../meshes/visual/link_0.stl
- link link_9: geometry visual mesh filename=../meshes/visual/link_1.stl
- link palm_link: geometry visual mesh filename=../meshes/visual/base_link.stl
